File: vin.kicad_sch (KiCad schematic)
At the start: 7 parts, among them J4 USB4105, U14 D5V0H1B2LP

Commit message: more pcb work, bom work
Parts:
- removed F1: Fuse, Fuse:Fuse_0805_2012Metric, symbol Device:Fuse
- C106: DigiKey_PN (none) -> 490-14603-1-ND; MPN (none) -> GRM155R71E104KE14J; Rating 10V/20% -> 25V/20%
- J4: DigiKey_PN (none) -> 2073-USB4105-GF-ACT-ND; MPN (none) -> USB4105-GF-A
- R41, R43: DigiKey_PN (none) -> 311-5.10KLRCT-ND; MPN (none) -> RC0402FR-075K1L
- U14: DigiKey_PN (none) -> D5V0H1B2LP-7BDICT-ND; MPN (none) -> D5V0H1B2LP-7B
Connections:
- net VBUS_VIN_R is gone; now on net VSYS_5V: J4.A4 (VBUS), J4.A9 (VBUS), J4.B4 (VBUS), J4.B9 (VBUS), U14.1
Changed lines of the file:
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@@
     (stroke (width 0) (type default) (color 0 0 0 0))
   )
-  (wire (pts (xy 80.01 55.88) (xy 88.9 55.88))
+  (wire (pts (xy 80.01 55.88) (xy 100.33 55.88))
     (stroke (width 0) (type default) (color 0 0 0 0))
   )
@@
   )
   (wire (pts (xy 52.07 63.5) (xy 45.72 63.5))
-    (stroke (width 0) (type default) (color 0 0 0 0))
-  )
-  (wire (pts (xy 96.52 55.88) (xy 100.33 55.88))
     (stroke (width 0) (type default) (color 0 0 0 0))
   )
@@
   )
   (label "VSYS_5V" (at 29.21 19.05 0)
-    (effects (font (size 1.27 1.27)) (justify left bottom))
-  )
-  (label "VBUS_VIN_R" (at 52.07 55.88 0)
     (effects (font (size 1.27 1.27)) (justify left bottom))
   )
@@
       (effects (font (size 1.27 1.27)) hide)
     )
-    (property "Rating" "10V/20%" (id 4) (at 106.68 66.04 0)
+    (property "Rating" "25V/20%" (id 4) (at 106.68 66.04 0)
       (effects (font (size 0.762 0.762)))
+    )
+    (property "DigiKey_PN" "490-14603-1-ND" (id 5) (at 100.33 62.23 0)
+      (effects (font (size 1.27 1.27)) hide)
+    )
+    (property "MPN" "GRM155R71E104KE14J" (id 6) (at 100.33 62.23 0)
+      (effects (font (size 1.27 1.27)) hide)
     )
     (pin "1")
@@
       (effects (font (size 0.762 0.762)))
     )
+    (property "DigiKey_PN" "311-5.10KLRCT-ND" (id 5) (at 52.07 69.85 0)
+      (effects (font (size 1.27 1.27)) hide)
+    )
+    (property "MPN" "RC0402FR-075K1L" (id 6) (at 52.07 69.85 0)
+      (effects (font (size 1.27 1.27)) hide)
+    )
     (pin "1")
     (pin "2")
@@
     )
     (property "Datasheet" "https://www.usb.org/sites/default/files/documents/usb_type-c.zip" (id 3) (at 34.29 71.12 0)
+      (effects (font (size 1.27 1.27)) hide)
+    )
+    (property "DigiKey_PN" "2073-USB4105-GF-ACT-ND" (id 4) (at 30.48 71.12 0)
+      (effects (font (size 1.27 1.27)) hide)
+    )
+    (property "MPN" "USB4105-GF-A" (id 5) (at 30.48 71.12 0)
       (effects (font (size 1.27 1.27)) hide)
     )
@@
       (effects (font (size 0.762 0.762)))
     )
+    (property "DigiKey_PN" "311-5.10KLRCT-ND" (id 5) (at 62.23 69.85 0)
+      (effects (font (size 1.27 1.27)) hide)
+    )
+    (property "MPN" "RC0402FR-075K1L" (id 6) (at 62.23 69.85 0)
+      (effects (font (size 1.27 1.27)) hide)
+    )
     (pin "1")
     (pin "2")
@@
     (pin "1")
   )
-  (symbol (lib_id "Device:Fuse") (at 92.71 55.88 90) (unit 1)
-    (in_bom yes) (on_board yes)
-    (property "Reference" "F1" (id 0) (at 92.71 49.53 90))
-    (property "Value" "Fuse" (id 1) (at 92.71 52.07 90))
-    (property "Footprint" "Fuse:Fuse_0805_2012Metric" (id 2) (at 92.71 57.658 90)
-      (effects (font (size 1.27 1.27)) hide)
-    )
-    (property "Datasheet" "~" (id 3) (at 92.71 55.88 0)
-      (effects (font (size 1.27 1.27)) hide)
-    )
-    (property "Rating" "3A" (id 4) (at 92.71 58.42 90)
-      (effects (font (size 0.762 0.762)))
-    )
-    (pin "1")
-    (pin "2")
-  )
   (symbol (lib_id "qsbc-zero:D5V0H1B2LP") (at 81.28 68.58 270) (unit 1)
     (in_bom yes) (on_board yes) (fields_autoplaced)
@@
       (effects (font (size 1.27 1.27)) hide)
     )
+    (property "DigiKey_PN" "D5V0H1B2LP-7BDICT-ND" (id 4) (at 81.28 68.58 0)
+      (effects (font (size 1.27 1.27)) hide)
+    )
+    (property "MPN" "D5V0H1B2LP-7B" (id 5) (at 81.28 68.58 0)
+      (effects (font (size 1.27 1.27)) hide)
+    )
