File: imx6ull_power.kicad_sch (KiCad schematic)
At the start: 20 parts, among them U1 MX6UL-VM

Commit message: more pcb work, bom work
Parts:
- C41, C57, C62: DigiKey_PN (none) -> 490-7611-1-ND; MPN (none) -> GRM188R60J226MEA0D
- C42, C43: DigiKey_PN (none) -> 1276-1482-1-ND; MPN (none) -> CL05A475MP5NRNC; Rating 6.3V/20% -> 10V/20%
- C44, C45, C46, C47, C48, C49, C51, C52, C54, C58, C59, C61: DigiKey_PN (none) -> 490-10392-1-ND; MPN (none) -> GRM033C80J224KE90D
- C55, C60: DigiKey_PN (none) -> 490-GRM155R60J106ME05DCT-ND; MPN (none) -> GRM155R60J106ME05D
- U1: DigiKey_PN (none) -> 568-14995-ND; MPN (none) -> MCIMX6Y2DVM09AB
Changed lines of the file:
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@@
       (effects (font (size 0.762 0.762)))
+    )
+    (property "DigiKey_PN" "490-10392-1-ND" (id 5) (at 250.19 114.3 0)
+      (effects (font (size 1.27 1.27)) hide)
+    )
+    (property "MPN" "GRM033C80J224KE90D" (id 6) (at 250.19 114.3 0)
+      (effects (font (size 1.27 1.27)) hide)
     )
     (pin "1")
@@
       (effects (font (size 0.762 0.762)))
     )
+    (property "DigiKey_PN" "490-10392-1-ND" (id 5) (at 300.99 114.3 0)
+      (effects (font (size 1.27 1.27)) hide)
+    )
+    (property "MPN" "GRM033C80J224KE90D" (id 6) (at 300.99 114.3 0)
+      (effects (font (size 1.27 1.27)) hide)
+    )
     (pin "1")
     (pin "2")
@@
       (effects (font (size 0.762 0.762)))
     )
+    (property "DigiKey_PN" "490-10392-1-ND" (id 5) (at 275.59 114.3 0)
+      (effects (font (size 1.27 1.27)) hide)
+    )
+    (property "MPN" "GRM033C80J224KE90D" (id 6) (at 275.59 114.3 0)
+      (effects (font (size 1.27 1.27)) hide)
+    )
     (pin "1")
     (pin "2")
@@
       (effects (font (size 1.27 1.27)) hide)
     )
-    (property "Rating" "6.3V/20%" (id 4) (at 129.54 109.22 0)
-      (effects (font (size 0.762 0.762)))
+    (property "Rating" "10V/20%" (id 4) (at 129.54 109.22 0)
+      (effects (font (size 0.762 0.762)))
+    )
+    (property "DigiKey_PN" "1276-1482-1-ND" (id 5) (at 124.46 105.41 0)
+      (effects (font (size 1.27 1.27)) hide)
+    )
+    (property "MPN" "CL05A475MP5NRNC" (id 6) (at 124.46 105.41 0)
+      (effects (font (size 1.27 1.27)) hide)
     )
     (pin "1")
@@
       (effects (font (size 1.27 1.27)) hide)
     )
-    (property "Rating" "6.3V/20%" (id 4) (at 118.11 137.16 0)
-      (effects (font (size 0.762 0.762)))
+    (property "Rating" "10V/20%" (id 4) (at 118.11 137.16 0)
+      (effects (font (size 0.762 0.762)))
+    )
+    (property "DigiKey_PN" "1276-1482-1-ND" (id 5) (at 113.03 133.35 0)
+      (effects (font (size 1.27 1.27)) hide)
+    )
+    (property "MPN" "CL05A475MP5NRNC" (id 6) (at 113.03 133.35 0)
+      (effects (font (size 1.27 1.27)) hide)
     )
     (pin "1")
@@
       (effects (font (size 0.762 0.762)))
     )
+    (property "DigiKey_PN" "490-7611-1-ND" (id 5) (at 113.03 105.41 0)
+      (effects (font (size 1.27 1.27)) hide)
+    )
+    (property "MPN" "GRM188R60J226MEA0D" (id 6) (at 113.03 105.41 0)
+      (effects (font (size 1.27 1.27)) hide)
+    )
     (pin "1")
     (pin "2")
@@
       (effects (font (size 0.762 0.762)))
     )
+    (property "DigiKey_PN" "490-10392-1-ND" (id 5) (at 250.19 153.67 0)
+      (effects (font (size 1.27 1.27)) hide)
+    )
+    (property "MPN" "GRM033C80J224KE90D" (id 6) (at 250.19 153.67 0)
+      (effects (font (size 1.27 1.27)) hide)
+    )
     (pin "1")
     (pin "2")
@@
     (property "Rating" "6.3V/20%" (id 4) (at 293.37 118.11 0)
       (effects (font (size 0.762 0.762)))
+    )
+    (property "DigiKey_PN" "490-7611-1-ND" (id 5) (at 288.29 114.3 0)
+      (effects (font (size 1.27 1.27)) hide)
+    )
+    (property "MPN" "GRM188R60J226MEA0D" (id 6) (at 288.29 114.3 0)
+      (effects (font (size 1.27 1.27)) hide)
     )
     (pin "1")
@@
       (effects (font (size 0.762 0.762)))
     )
+    (property "DigiKey_PN" "490-GRM155R60J106ME05DCT-ND" (id 5) (at 300.99 153.67 0)
+      (effects (font (size 1.27 1.27)) hide)
+    )
+    (property "MPN" "GRM155R60J106ME05D" (id 6) (at 300.99 153.67 0)
+      (effects (font (size 1.27 1.27)) hide)
+    )
     (pin "1")
     (pin "2")
@@
       (effects (font (size 0.762 0.762)))
     )
+    (property "DigiKey_PN" "490-10392-1-ND" (id 5) (at 124.46 133.35 0)
+      (effects (font (size 1.27 1.27)) hide)
+    )
+    (property "MPN" "GRM033C80J224KE90D" (id 6) (at 124.46 133.35 0)
+      (effects (font (size 1.27 1.27)) hide)
+    )
     (pin "1")
     (pin "2")
@@
     (property "Rating" "6.3V/20%" (id 4) (at 318.77 118.11 0)
       (effects (font (size 0.762 0.762)))
+    )
+    (property "DigiKey_PN" "490-10392-1-ND" (id 5) (at 313.69 114.3 0)
+      (effects (font (size 1.27 1.27)) hide)
+    )
+    (property "MPN" "GRM033C80J224KE90D" (id 6) (at 313.69 114.3 0)
+      (effects (font (size 1.27 1.27)) hide)
     )
     (pin "1")
@@
     (property "Datasheet" "" (id 3) (at 212.344 115.824 0)
       (effects (font (size 1.524 1.524)))
+    )
+    (property "DigiKey_PN" "568-14995-ND" (id 4) (at 199.39 86.36 0)
+      (effects (font (size 1.27 1.27)) hide)
+    )
+    (property "MPN" "MCIMX6Y2DVM09AB" (id 5) (at 199.39 86.36 0)
+      (effects (font (size 1.27 1.27)) hide)
     )
     (pin "A1")
@@
       (effects (font (size 0.762 0.762)))
     )
+    (property "DigiKey_PN" "490-10392-1-ND" (id 5) (at 135.89 105.41 0)
+      (effects (font (size 1.27 1.27)) hide)
+    )
+    (property "MPN" "GRM033C80J224KE90D" (id 6) (at 135.89 105.41 0)
+      (effects (font (size 1.27 1.27)) hide)
+    )
     (pin "1")
     (pin "2")
@@
       (effects (font (size 0.762 0.762)))
     )
+    (property "DigiKey_PN" "490-10392-1-ND" (id 5) (at 262.89 114.3 0)
+      (effects (font (size 1.27 1.27)) hide)
+    )
+    (property "MPN" "GRM033C80J224KE90D" (id 6) (at 262.89 114.3 0)
+      (effects (font (size 1.27 1.27)) hide)
+    )
     (pin "1")
     (pin "2")
@@
       (effects (font (size 0.762 0.762)))
     )
+    (property "DigiKey_PN" "490-10392-1-ND" (id 5) (at 148.59 143.51 0)
+      (effects (font (size 1.27 1.27)) hide)
+    )
+    (property "MPN" "GRM033C80J224KE90D" (id 6) (at 148.59 143.51 0)
+      (effects (font (size 1.27 1.27)) hide)
+    )
     (pin "1")
     (pin "2")
@@
       (effects (font (size 0.762 0.762)))
     )
+    (property "DigiKey_PN" "490-10392-1-ND" (id 5) (at 262.89 153.67 0)
+      (effects (font (size 1.27 1.27)) hide)
+    )
+    (property "MPN" "GRM033C80J224KE90D" (id 6) (at 262.89 153.67 0)
+      (effects (font (size 1.27 1.27)) hide)
+    )
     (pin "1")
     (pin "2")
@@
       (effects (font (size 0.762 0.762)))
     )
+    (property "DigiKey_PN" "490-7611-1-ND" (id 5) (at 326.39 114.3 0)
+      (effects (font (size 1.27 1.27)) hide)
+    )
+    (property "MPN" "GRM188R60J226MEA0D" (id 6) (at 326.39 114.3 0)
+      (effects (font (size 1.27 1.27)) hide)
+    )
     (pin "1")
     (pin "2")
@@
       (effects (font (size 0.762 0.762)))
     )
+    (property "DigiKey_PN" "490-GRM155R60J106ME05DCT-ND" (id 5) (at 275.59 153.67 0)
+      (effects (font (size 1.27 1.27)) hide)
+    )
+    (property "MPN" "GRM155R60J106ME05D" (id 6) (at 275.59 153.67 0)
+      (effects (font (size 1.27 1.27)) hide)
+    )
     (pin "1")
     (pin "2")
@@
       (effects (font (size 0.762 0.762)))
     )
+    (property "DigiKey_PN" "490-10392-1-ND" (id 5) (at 288.29 153.67 0)
+      (effects (font (size 1.27 1.27)) hide)
+    )
+    (property "MPN" "GRM033C80J224KE90D" (id 6) (at 288.29 153.67 0)
+      (effects (font (size 1.27 1.27)) hide)
+    )
     (pin "1")
     (pin "2")
@@
       (effects (font (size 0.762 0.762)))
     )
-    (pin "1")
+    (property "DigiKey_PN" "490-10392-1-ND" (id 5) (at 148.59 105.41 0)
+      (effects (font (size 1.27 1.27)) hide)
+    )
+    (property "MPN" "GRM033C80J224KE90D" (id 6) (at 148.59 105.41 0)
+      (effects (font (size 1.27 1.27)) hide)
+    )
+    (pin "1")

Commit message: add basic readme, rev 1 of pcb
Parts:
- C41, C57, C62: DigiKey_PN 490-7611-1-ND -> 1276-1274-1-ND; MPN GRM188R60J226MEA0D -> CL10A226MP8NUNE; Rating 6.3V/20% -> 10V/20%
Connections:
- net SNVS_3V3 renamed SNVS_3V
Changed lines of the file:
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@@
     (effects (font (size 1.27 1.27)) (justify right bottom))
   )
-  (label "SNVS_3V3" (at 137.16 137.16 0)
+  (label "SNVS_3V" (at 137.16 137.16 0)
     (effects (font (size 1.27 1.27)) (justify left bottom))
   )
@@
     (effects (font (size 1.27 1.27)) (justify left bottom))
   )
-  (label "SNVS_3V3" (at 36.83 33.02 0)
+  (label "SNVS_3V" (at 36.83 33.02 0)
     (effects (font (size 1.27 1.27)) (justify left bottom))
   )
@@
     (effects (font (size 1.27 1.27)) (justify right))
   )
-  (hierarchical_label "SNVS_3V3" (shape input) (at 34.29 33.02 180)
+  (hierarchical_label "SNVS_3V" (shape input) (at 34.29 33.02 180)
     (effects (font (size 1.27 1.27)) (justify right))
   )
@@
       (effects (font (size 1.27 1.27)) hide)
     )
-    (property "Rating" "6.3V/20%" (id 4) (at 118.11 109.22 0)
-      (effects (font (size 0.762 0.762)))
-    )
-    (property "DigiKey_PN" "490-7611-1-ND" (id 5) (at 113.03 105.41 0)
-      (effects (font (size 1.27 1.27)) hide)
-    )
-    (property "MPN" "GRM188R60J226MEA0D" (id 6) (at 113.03 105.41 0)
+    (property "Rating" "10V/20%" (id 4) (at 118.11 109.22 0)
+      (effects (font (size 0.762 0.762)))
+    )
+    (property "DigiKey_PN" "1276-1274-1-ND" (id 5) (at 113.03 105.41 0)
+      (effects (font (size 1.27 1.27)) hide)
+    )
+    (property "MPN" "CL10A226MP8NUNE" (id 6) (at 113.03 105.41 0)
       (effects (font (size 1.27 1.27)) hide)
     )
@@
       (effects (font (size 1.27 1.27)) hide)
     )
-    (property "Rating" "6.3V/20%" (id 4) (at 293.37 118.11 0)
-      (effects (font (size 0.762 0.762)))
-    )
-    (property "DigiKey_PN" "490-7611-1-ND" (id 5) (at 288.29 114.3 0)
-      (effects (font (size 1.27 1.27)) hide)
-    )
-    (property "MPN" "GRM188R60J226MEA0D" (id 6) (at 288.29 114.3 0)
+    (property "Rating" "10V/20%" (id 4) (at 293.37 118.11 0)
+      (effects (font (size 0.762 0.762)))
+    )
+    (property "DigiKey_PN" "1276-1274-1-ND" (id 5) (at 288.29 114.3 0)
+      (effects (font (size 1.27 1.27)) hide)
+    )
+    (property "MPN" "CL10A226MP8NUNE" (id 6) (at 288.29 114.3 0)
       (effects (font (size 1.27 1.27)) hide)
     )
@@
       (effects (font (size 1.27 1.27)) hide)
     )
-    (property "Rating" "6.3V/20%" (id 4) (at 331.47 118.11 0)
-      (effects (font (size 0.762 0.762)))
-    )
-    (property "DigiKey_PN" "490-7611-1-ND" (id 5) (at 326.39 114.3 0)
-      (effects (font (size 1.27 1.27)) hide)
-    )
-    (property "MPN" "GRM188R60J226MEA0D" (id 6) (at 326.39 114.3 0)
-      (effects (font (size 1.27 1.27)) hide)
-    )
+    (property "Rating" "10V/20%" (id 4) (at 331.47 118.11 0)
+      (effects (font (size 0.762 0.762)))
+    )
+    (property "DigiKey_PN" "1276-1274-1-ND" (id 5) (at 326.39 114.3 0)
+      (effects (font (size 1.27 1.27)) hide)
+    )
+    (property "MPN" "CL10A226MP8NUNE" (id 6) (at 326.39 114.3 0)
+      (effects (font (size 1.27 1.27)) hide)
+    )
