File: qsbc-zero.kicad_pcb (KiCad board)
At the start: 4 copper layers, 80 x 80 mm, 276 parts, among them J1 Micro_SD_Card_Det1, J11 Conn_01x02_Male, J2 USB4105, J3 USB-A-S-F-B-VU, J4 USB4105, J5 Conn_02x18_Odd_Even, J6 J1B1211CCD, J7 Conn_01x06_Male, J8 Conn_02x16_Odd_Even, Q2 2SK3019, Q3 2SK3019, Q4 2SK3019, SW2 SW_Push, U1 MX6UL-VM, U11 TPD4EUSB30, U12 74LVC1G04, U13 D5V0H1B2LP, U14 D5V0H1B2LP, U18 DP83825, U19 TLV62569DDC, U2 TLV62569DDC, U20 TLV62569DDC, U21 TPS7A0333DBVR, U24 NCP164CSNADJT1G, U25 TPD4EUSB30, U26 TPD4EUSB30, U27 TPD4EUSB30, U28 LMV331, U3 MT41K256M16, U4 TUSB320, U5 AP22814AW5, U6 TPD4EUSB30, U7 D5V0H1B2LP, U8 D5V0H1B2LP, U9 W25Q32JVZP, Y1 24Mhz, Y2 32.768kHz

Commit message: more pcb work, bom work
Parts:
- removed F1: Fuse, Fuse:Fuse_0805_2012Metric
- removed Q4: 2SK3019, Package_TO_SOT_SMD:SOT-416
- removed U24: NCP164CSNADJT1G, Package_SO:TSOP-5_1.65x3.05mm_P0.95mm
- added JP1: Jumper_2_Open, Jumper:SolderJumper-2_P1.3mm_Open_RoundedPad1.0x1.5mm, F.Cu at (164.2, 101.3)
- added JP2: Jumper_2_Open, Jumper:SolderJumper-2_P1.3mm_Open_RoundedPad1.0x1.5mm, F.Cu at (168.6, 101.3)
- added Q1: SSM3K15ACT, Package_TO_SOT_SMD:SOT-883, F.Cu at (164.9, 127.9)
- added R21: 10K, Resistor_SMD:R_0402_1005Metric, F.Cu at (190.0, 95.3)
- added R22: 0R, Resistor_SMD:R_0402_1005Metric, F.Cu at (190.0, 91.9)
- added TP4: TestPoint, TestPoint:TestPoint_Pad_D1.0mm, F.Cu at (161.8, 116.9)
- added U10: AP7330, qsbc-zero:SOT-753, F.Cu at (199.7, 84.2)
- C53, C66, C81: footprint Capacitor_SMD:C_0201_0603Metric -> Capacitor_SMD:C_0402_1005Metric
- D1: value LED -> LED_GREEN
- D2: value LED -> LED_ORANGE
- J11: footprint Connector_PinHeader_2.54mm:PinHeader_1x02_P2.54mm_Vertical_SMD_Pin1Left -> Connector_PinHeader_2.54mm:PinHeader_1x02_P2.54mm_Vertical
- Q2, Q3: value 2SK3019 -> SSM3K15ACT; footprint Package_TO_SOT_SMD:SOT-416 -> Package_TO_SOT_SMD:SOT-883
- R122: value 200K -> 316K
- R125: value 93.1K -> 210K
- R4: footprint Capacitor_SMD:C_0201_0603Metric -> Resistor_SMD:R_0201_0603Metric
- R5: footprint Resistor_SMD:R_0402_1005Metric -> Resistor_SMD:R_0201_0603Metric
- R9: footprint Capacitor_SMD:C_0402_1005Metric -> Resistor_SMD:R_0402_1005Metric
- U5: value AP22814AW5 -> AP22811B
- U9: value W25Q32JVZP -> W25Q256JWPIQ
- moved R8 73.5 mm to (172.7, 134.7), turned to -90 degrees
- moved C3 72.3 mm to (169.1, 138.1), turned to -90 degrees
- moved R6 71.8 mm to (171.7, 134.7), turned to -90 degrees
- moved Q3 71.7 mm to (199.4, 81.1), turned to 90 degrees
- moved R48 67.5 mm to (171.6, 131.8)
- moved R26 66.5 mm to (167.1, 134.9), turned to 180 degrees
- moved R25 64.6 mm to (167.6, 133.4), turned to -90 degrees
- moved D6 64.4 mm to (168.0, 140.9)
- moved C8 63.4 mm to (169.6, 133.4), turned to -90 degrees
- moved C1 61.5 mm to (170.6, 134.7), turned to -90 degrees
- moved C6 60.9 mm to (168.6, 133.4), turned to -90 degrees
- moved R23 59.8 mm to (168.0, 138.1), turned to 90 degrees
- moved TP17 59.0 mm to (170.8, 130.0)
- moved R16 58.3 mm to (170.1, 138.1), turned to -90 degrees
- moved C7 55.5 mm to (168.1, 130.9)
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Connections:
- C14 pad 1: /Power/VDD_SNVS_3V3 -> VDD_SNVS_3V3
- C20 pad 2: Net-(C20-Pad2) -> GND
- C22 pad 2: Net-(C20-Pad2) -> GND
- C82 pad 1: /USB/VBUS_1 -> VSYS_5V
- D7 pad 2: /Power/VDD_SNVS_3V3 -> VDD_SNVS_3V3
- J1 pad 10: GND -> /Peripherals/SD1_CD
- J4 pad A4: /VIN/VBUS_VIN_R -> VSYS_5V
- J4 pad A9: /VIN/VBUS_VIN_R -> VSYS_5V
- J4 pad B4: /VIN/VBUS_VIN_R -> VSYS_5V
- J4 pad B9: /VIN/VBUS_VIN_R -> VSYS_5V
- J5 pad 1: VSYS_5V -> GND
- J5 pad 10: /Peripherals/GPIO1_IO04 -> /Peripherals/GPIO1_IO06
- J5 pad 11: /Peripherals/GPIO1_IO05 -> GND
- J5 pad 12: /Peripherals/GPIO1_IO07 -> GND
- J5 pad 13: /Peripherals/GPIO1_IO03 -> GPIO1_IO21
- J5 pad 14: /Peripherals/GPIO1_IO06 -> GPIO1_IO20
- J5 pad 15: GND -> GPIO1_IO25
- J5 pad 16: GND -> GPIO1_IO24
- J5 pad 17: GPIO1_IO21 -> GPIO1_IO29
- J5 pad 18: GPIO1_IO20 -> GPIO1_IO28
- J5 pad 19: GPIO1_IO25 -> GPIO1_IO30
- J5 pad 2: DCDC_3V3 -> GND
- J5 pad 20: GPIO1_IO24 -> GPIO1_IO11
- J5 pad 21: GPIO1_IO29 -> GPIO1_IO13
- J5 pad 22: GPIO1_IO28 -> GPIO1_IO14
- J5 pad 23: GPIO1_IO30 -> /Peripherals/GPIO1_IO09
- J5 pad 24: GPIO1_IO11 -> GPIO1_IO10
- J5 pad 25: GPIO1_IO13 -> GND
- J5 pad 26: GPIO1_IO14 -> GND
- J5 pad 27: /Peripherals/GPIO1_IO09 -> GPIO1_IO22
- J5 pad 28: GPIO1_IO10 -> GPIO1_IO26
- J5 pad 29: GND -> GPIO1_IO23
- J5 pad 3: VSYS_5V -> GPIO1_IO15
- J5 pad 30: GND -> GPIO1_IO27
- J5 pad 31: GPIO1_IO22 -> GND
- J5 pad 32: GPIO1_IO26 -> GPIO1_IO31
- J5 pad 33: GPIO1_IO23 -> VSYS_5V
- J5 pad 34: GPIO1_IO27 -> DCDC_3V3
- J5 pad 35: GND -> VSYS_5V
- J5 pad 36: GPIO1_IO31 -> DCDC_3V3
- J5 pad 4: DCDC_3V3 -> GPIO1_IO12
- J5 pad 5: GND -> /Peripherals/GPIO1_IO08
- J5 pad 6: GND -> /Peripherals/GPIO1_IO04
- J5 pad 7: GPIO1_IO15 -> /Peripherals/GPIO1_IO05
- J5 pad 8: GPIO1_IO12 -> /Peripherals/GPIO1_IO07
- J5 pad 9: /Peripherals/GPIO1_IO08 -> /Peripherals/GPIO1_IO03
- Q2 pad 1: Net-(Q2-Pad1) -> PMIC_STBY_REQ
- Q2 pad 2: GPIO_DVFS -> Net-(R110-Pad1)
- Q2 pad 3: Net-(Q2-Pad3) -> Net-(R118-Pad2)
- Q3 pad 1: Net-(Q2-Pad1) -> SD1_VSELECT
- Q3 pad 2: PMIC_STBY_REQ -> Net-(R122-Pad2)
- Q3 pad 3: Net-(Q3-Pad3) -> Net-(R125-Pad2)
- R110 pad 1: Net-(Q2-Pad1) -> Net-(R110-Pad1)
- R116 pad 2: Net-(Q2-Pad3) -> Net-(R116-Pad2)
- R118 pad 2: Net-(Q3-Pad3) -> Net-(R118-Pad2)
- R122 pad 2: Net-(Q4-Pad1) -> Net-(R122-Pad2)
- R123 pad 1: Net-(Q4-Pad1) -> Net-(R122-Pad2)
- R125 pad 2: Net-(Q4-Pad3) -> Net-(R125-Pad2)
- R139 pad 2: /Control/BOOT_MODE1 -> Net-(R139-Pad2)
- R140 pad 2: /Control/BOOT_MODE0 -> Net-(R140-Pad2)
- R58 pad 1: Net-(C20-Pad2) -> GND
- R61 pad 2: Net-(Q2-Pad1) -> Net-(R110-Pad1)
- U1 pad D3: unconnected-(U1-PadD3) -> /Peripherals/SD1_CD_R
- U1 pad F1: unconnected-(U1-PadF1) -> /DDR/DRAM_SDCKE1
- U14 pad 1: /VIN/VBUS_VIN_R -> VSYS_5V
- U18 pad 26: (no net) -> GND
- U18 pad 27: (no net) -> GND
- U18 pad 28: (no net) -> GND
- U18 pad 29: (no net) -> GND
- U18 pad 30: (no net) -> GND
- U2 pad 6: Net-(Q2-Pad1) -> Net-(R110-Pad1)
- U21 pad 5: /Power/VDD_SNVS_3V3 -> VDD_SNVS_3V3
- U27 pad 4: unconnected-(U27-Pad4) -> /Peripherals/SD1_CD
- U27 pad 7: unconnected-(U27-Pad4) -> /Peripherals/SD1_CD
Routing:
- net ~{WDOG}: track 0.57 -> 162.9 mm, vias 1 -> 4
- net VSYS_5V: track 11.1 -> 157.7 mm, vias 8 -> 12
- net /Power/PG_3V3: track 0.00 -> 120.9 mm, vias 0 -> 1
- net GND: track 238.5 -> 304.1 mm, vias 135 -> 167
- net GPIO_DVFS: track 28.7 -> 0.00 mm, vias 1 -> 0
- net /Ethernet/RJ45_LED_Y: track 0.00 -> 22.5 mm
- net /Peripherals/SD1_CD: track 0.00 -> 22.1 mm, vias 0 -> 2
- net Net-(C3-Pad1): track 0.00 -> 18.7 mm, vias 0 -> 3
- net /Ethernet/ENET1_TX_DATA1: track 0.00 -> 17.3 mm, vias 0 -> 2
- net /Ethernet/RJ45_LED_G: track 0.00 -> 15.9 mm, vias 0 -> 1
- net /Control/BOOT_MODE0: track 16.4 -> 32.1 mm
- net /Control/BOOT_MODE1: track 15.7 -> 0.00 mm
- net /Ethernet/ENET1_TX_DATA0: track 0.00 -> 15.4 mm, vias 0 -> 2
- net ~{USB1_INT}: track 21.8 -> 36.3 mm, vias 1 -> 2
- net SNVS_3V3: track 2.28 -> 16.6 mm
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- added copper zone on In2.Cu, net DCDC_3V3
- removed copper zone on F.Cu, net /VIN/VBUS_VIN_R
- removed copper zone on In2.Cu, net GND

Commit message: add basic readme, rev 1 of pcb
Parts:
- removed C114, C115, C124: 4.7uF, Capacitor_SMD:C_0402_1005Metric
- removed C116, C117, C118, C119, C120, C121: 10uF, Capacitor_SMD:C_0402_1005Metric
- removed C125: 0.1uF, Capacitor_SMD:C_0402_1005Metric
- removed D6, D7, D8: PMEG3010AESBYL, Diode_SMD:D_SOD-323F
- removed Q1, Q2, Q3: SSM3K15ACT, Package_TO_SOT_SMD:SOT-883
- removed R110, R111, R117, R123, R124, R135, R60: 100K, Resistor_SMD:R_0402_1005Metric
- removed R116: 953K, Resistor_SMD:R_0402_1005Metric
- removed R118: 91K, Resistor_SMD:R_0402_1005Metric
- removed R119, R120, R126, R127, R48: 0R, Resistor_SMD:R_0603_1608Metric
- removed R122: 316K, Resistor_SMD:R_0402_1005Metric
- removed R125: 210K, Resistor_SMD:R_0402_1005Metric
- removed R136: 10K, Resistor_SMD:R_0402_1005Metric
- removed R137: 21K, Resistor_SMD:R_0402_1005Metric
- removed R142: 0R, Resistor_SMD:R_0402_1005Metric
- removed R56: 1K, Resistor_SMD:R_0402_1005Metric
- removed R57, R58: 1.5K, Resistor_SMD:R_0402_1005Metric
- removed R59: 124K, Resistor_SMD:R_0402_1005Metric
- removed R61: 133K, Resistor_SMD:R_0402_1005Metric
- removed SW2: SW_Push, Button_Switch_THT:SW_Tactile_SPST_Angled_PTS645Vx58-2LFS
- removed TP1, TP15, TP16, TP17, TP18, TP2, TP20, TP23, TP24, TP27, TP28: TestPoint, TestPoint:TestPoint_Pad_D1.0mm
- removed U10: AP7330, qsbc-zero:SOT-753
- removed U19, U20: TLV62569DDC, Package_TO_SOT_SMD:SOT-23-6
- removed U21: TPS7A0333DBVR, Package_TO_SOT_SMD:SOT-23-5
- removed U28: LMV331, Package_TO_SOT_SMD:SOT-23-5
- added C11: 22uF, Capacitor_SMD:C_0603_1608Metric, F.Cu at (160.2, 131.6)
- added C12: 22uF, Capacitor_SMD:C_0603_1608Metric, F.Cu at (161.8, 131.6)
- added C16: 10uF, Capacitor_SMD:C_0402_1005Metric, F.Cu at (159.9, 119.2)
- added C17: 4.7uF, Capacitor_SMD:C_0402_1005Metric, F.Cu at (156.8, 129.2)
- added C83: 0.47uF, Capacitor_SMD:C_0402_1005Metric, F.Cu at (157.9, 130.8)
- added C84: 10uF, Capacitor_SMD:C_0402_1005Metric, F.Cu at (150.7, 130.6)
- added C85: 0.22uF, Capacitor_SMD:C_0201_0603Metric, F.Cu at (176.9, 108.6)
- added C86: 0.22uF, Capacitor_SMD:C_0201_0603Metric, F.Cu at (185.6, 124.7)
- added C87: 4.7uF, Capacitor_SMD:C_0402_1005Metric, B.Cu at (156.3, 126.7)
- added C88: 1uF, Capacitor_SMD:C_0402_1005Metric, F.Cu at (156.3, 127.7)
- added C89: 4.7uF, Capacitor_SMD:C_0402_1005Metric, B.Cu at (160.8, 122.0)
- added C90: 1uF, Capacitor_SMD:C_0402_1005Metric, F.Cu at (156.7, 122.0)
- added C91: 4.7uF, Capacitor_SMD:C_0402_1005Metric, B.Cu at (161.9, 122.0)
- added C96: 1uF, Capacitor_SMD:C_0402_1005Metric, B.Cu at (165.2, 124.0)
- added D3: LED_YELLOW, LED_SMD:LED_0603_1608Metric, F.Cu at (211.4, 67.9)
- added J10: Conn_02x18_Odd_Even, Connector_PinHeader_2.54mm:PinHeader_2x18_P2.54mm_Vertical, F.Cu at (219.7, 75.4)
- added J9: Conn_01x02_Male, Connector_PinHeader_2.54mm:PinHeader_1x02_P2.54mm_Vertical, F.Cu at (150.2, 133.0)
- added SW1: SW_Push, Button_Switch_THT:SW_Tactile_SPST_Angled_PTS645Vx58-2LFS, F.Cu at (156.5, 68.7)
- added TP6: TestPoint, TestPoint:TestPoint_Pad_D1.0mm, B.Cu at (192.2, 95.5)
- C1: value 1uF -> 0.1uF
- C13, C14, C18: value 1uF -> 10uF
- C15: value 0.1uF -> 10uF
- C20: value 4.7uF -> 10uF
- C21: value 0.1uF -> 4.7uF
- C22: value 0.1uF -> 1uF; moved to B.Cu
- C3: value 0.22uF -> 10uF
- C5: value 4.7uF -> 0.1uF; moved to B.Cu
- C53: value 0.1uF -> 0.22uF; footprint Capacitor_SMD:C_0402_1005Metric -> Capacitor_SMD:C_0201_0603Metric
- C6, C8: value 10uF -> 1uF
- C7: value 10uF -> 2.2uF
- C9: moved to B.Cu
- J11: value Conn_01x02_Male -> Conn_01x09_Male; footprint Connector_PinHeader_2.54mm:PinHeader_1x02_P2.54mm_Vertical -> Connector_PinHeader_1.27mm:PinHeader_1x09_P1.27mm_Vertical
- J8: value Conn_02x16_Odd_Even -> Conn_01x09_Male; footprint Connector_PinHeader_2.54mm:PinHeader_2x16_P2.54mm_Vertical -> Connector_PinHeader_1.27mm:PinHeader_1x09_P1.27mm_Vertical
- L1, L2, L3: value 2.2uH -> 1uH; footprint Inductor_SMD:L_Vishay_IHLP-1212 -> Inductor_SMD:L_0603_1608Metric
- R23: value 0R -> 100K
- R24: value 499K -> 100K
- R25: value 442K -> 0R
- R26: value 100K -> 1K
- R6: value 10K -> 100K
- R7: value 1M -> 100K
- U2: value TLV62569DDC -> MC32PF1510A6EP; footprint Package_TO_SOT_SMD:SOT-23-6 -> Package_DFN_QFN:QFN-40-1EP_5x5mm_P0.4mm_EP3.8x3.8mm_ThermalVias
- U9: value W25Q256JWPIQ -> W25Q512JVEIQ
- moved R26 77.3 mm to (211.4, 71.6), turned to 90 degrees
- moved J8 66.3 mm to (153.4, 75.4), turned to 90 degrees
- moved C13 64.0 mm to (153.6, 125.8)
- moved C19 52.6 mm to (159.1, 122.1), turned to 90 degrees
- moved C14 50.0 mm to (152.6, 125.8), turned to 90 degrees
- moved C18 47.7 mm to (162.8, 117.9)
- moved C9 47.5 mm to (156.3, 125.0), turned to 180 degrees
- moved C15 46.9 mm to (159.9, 117.9), turned to 180 degrees
- moved J11 42.2 mm to (201.9, 75.4), turned to 90 degrees
- moved C22 37.1 mm to (156.3, 124.0), turned to 180 degrees
- moved C21 36.3 mm to (163.6, 122.1), turned to 90 degrees
- moved C20 32.4 mm to (162.8, 119.2), turned to 0 degrees
- moved R20 21.4 mm to (156.0, 81.6), turned to 0 degrees
- moved C3 20.3 mm to (150.7, 129.5), turned to 0 degrees
- moved C6 16.0 mm to (155.6, 124.0), turned to 180 degrees
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Connections:
- net /Peripherals/SD1_CD renamed SD1_CD
- C1 pad 1: ~{WDOG} -> /Power/LICELL
- C1 pad 2: Net-(C1-Pad2) -> GND
- C13 pad 1: VSYS_5V -> VDD_ARM_SOC_IN
- C14 pad 1: VDD_SNVS_3V3 -> VDD_ARM_SOC_IN
- C15 pad 1: Net-(C15-Pad1) -> DDR_1V35
- C18 pad 1: /Power/SD_3V3_1V8_R -> DCDC_3V3
- C19 pad 1: Net-(C15-Pad1) -> LDO2_3V3
- C20 pad 1: DDR_1V35 -> DCDC_3V3
- C21 pad 1: DDR_1V35 -> SD_3V3_1V8
- C21 pad 2: /DDR/VREFDDR -> GND
- C22 pad 1: /DDR/VREFDDR -> DDR_VREF
- C24 pad 1: /DDR/VREFDDR -> DDR_VREF
- C28 pad 1: /DDR/VREFDDR -> DDR_VREF
- C29 pad 1: /DDR/VREFDDR -> DDR_VREF
- C3 pad 1: Net-(C3-Pad1) -> /Power/LICELL
- C47 pad 1: SNVS_3V3 -> /SNVS_3V3
- C5 pad 1: VSYS_5V -> DCDC_3V3
- C53 pad 1: DCDC_3V3 -> LDO2_3V3
- C56 pad 1: DCDC_3V3 -> LDO2_3V3
- C6 pad 1: /Power/DCDC_3V3_R -> DDR_1V35
- C7 pad 1: /Power/DCDC_3V3_R -> VSYS_5V
- C8 pad 1: /Power/DCDC_3V3_R -> /Power/VCORE
- C9 pad 1: VSYS_5V -> /Power/VDIG
- J11 pad 1: Net-(C15-Pad1) -> DCDC_3V3
- J11 pad 2: GND -> I2C2_SCL
- J8 pad 1: GND -> DCDC_3V3
- J8 pad 2: GND -> /Power/PWRON
- J8 pad 3: /Peripherals/BT_CFG1[0] -> PMIC_ON_REQ
- J8 pad 4: /Peripherals/BT_CFG1[1] -> ~{POR}
- J8 pad 5: /Peripherals/BT_CFG1[2] -> /SNVS_3V3
- J8 pad 6: /Peripherals/BT_CFG1[3] -> /Power/PMIC_ONOFF
- J8 pad 7: /Peripherals/BT_CFG1[4] -> IMX6_ONOFF
- J8 pad 8: /Peripherals/BT_CFG1[5] -> PMIC_STBY_REQ
- J8 pad 9: /Peripherals/BT_CFG1[6] -> GND
- L1 pad 2: /Power/DCDC_3V3_R -> VDD_ARM_SOC_IN
- L2 pad 2: /Power/DDR_1V35_R -> DDR_1V35
- L3 pad 2: /Power/VDD_ARM_SOC_IN_R -> DCDC_3V3
- R139 pad 1: SNVS_3V3 -> /SNVS_3V3
- R140 pad 1: SNVS_3V3 -> /SNVS_3V3
- R16 pad 1: Net-(C3-Pad1) -> /SNVS_3V3
- R16 pad 2: GND -> ~{PMIC_INT}
- R23 pad 1: Net-(D6-Pad2) -> /SNVS_3V3
- R23 pad 2: Net-(C3-Pad1) -> ~{POR}
- R24 pad 1: VSYS_5V -> /Power/VSYS
- R24 pad 2: /Power/PG_3V3 -> /Power/PMIC_ONOFF
- R25 pad 1: /Power/DCDC_3V3_R -> /Power/PWRON
- R25 pad 2: Net-(R25-Pad2) -> PMIC_ON_REQ
- R26 pad 1: Net-(R25-Pad2) -> DCDC_3V3
- R26 pad 2: GND -> Net-(D3-Pad2)
- R6 pad 1: PMIC_ON_REQ -> DCDC_3V3
- R6 pad 2: Net-(C3-Pad1) -> ~{WDOG}
- R7 pad 1: Net-(C1-Pad2) -> /SNVS_3V3
- R7 pad 2: GND -> /Power/PWRON
- R8 pad 1: VSYS_5V -> /SNVS_3V3
- R8 pad 2: Net-(C3-Pad1) -> PMIC_STBY_REQ
- TP4 pad 1: GPIO_DVFS -> /Power/LDO1_1V8
- U1 pad A5: unconnected-(U1-PadA5) -> /Storage/ECSPI4_CS0
- U1 pad A6: unconnected-(U1-PadA6) -> /Storage/ECSPI4_MISO
- U1 pad A8: unconnected-(U1-PadA8) -> /Peripherals/LCD_CLK
- U1 pad B6: unconnected-(U1-PadB6) -> /Storage/ECSPI4_MOSI
- U1 pad B7: unconnected-(U1-PadB7) -> /Storage/ECSPI4_CS1
- U1 pad B8: unconnected-(U1-PadB8) -> /Peripherals/LCD_ENABLE
- U1 pad C6: unconnected-(U1-PadC6) -> /Storage/ECSPI4_SCLK
- U1 pad C9: unconnected-(U1-PadC9) -> /Peripherals/LCD_VSYNC
- U1 pad D1: SD1_VSELECT -> /Peripherals/SD1_VSELECT
- U1 pad D2: unconnected-(U1-PadD2) -> /Peripherals/LED_2
- U1 pad D9: unconnected-(U1-PadD9) -> /Peripherals/LCD_HSYNC
- U1 pad F2: unconnected-(U1-PadF2) -> I2C2_SDA
- U1 pad F3: unconnected-(U1-PadF3) -> I2C2_SCL
- U1 pad L13: DCDC_3V3 -> LDO2_3V3
- U1 pad M13: DCDC_3V3 -> LDO2_3V3
- U1 pad P12: SNVS_3V3 -> /SNVS_3V3
- U1 pad P4: /DDR/VREFDDR -> DDR_VREF
- U1 pad P8: /Control/JTAG_nSRST -> ~{POR}
- U1 pad R10: GPIO_DVFS -> ~{PMIC_INT}
- U1 pad R8: /Control/ONOFF -> IMX6_ONOFF
- U2 pad 1: /Power/PG_3V3 -> ~{WDOG}
- U2 pad 2: GND -> I2C4_SDA
- U2 pad 3: Net-(L3-Pad1) -> I2C4_SCL
- U2 pad 4: VSYS_5V -> DCDC_3V3
- U2 pad 5: /Power/ARM_SOC_PG -> GND
- U2 pad 6: Net-(R110-Pad1) -> /Power/PWRON
- U3 pad H1: /DDR/VREFDDR -> DDR_VREF
- U3 pad M8: /DDR/VREFDDR -> DDR_VREF
Routing:
- net /Power/PG_3V3: track 120.9 -> 0.00 mm, vias 1 -> 0
- net /SNVS_3V3: track 0.00 -> 117.6 mm, vias 0 -> 7
- net /Control/ONOFF: track 94.0 -> 0.00 mm, vias 1 -> 0
- net /Power/PMIC_ONOFF: track 0.00 -> 82.9 mm, vias 0 -> 1
- net ~{POR}: track 0.00 -> 74.7 mm, vias 0 -> 3
- net SD_3V3_1V8: track 6.16 -> 79.9 mm, vias 5 -> 4
- net DDR_VREF: track 0.00 -> 73.4 mm, vias 0 -> 4
- net /Power/PWRON: track 0.00 -> 71.3 mm, vias 0 -> 2
- net LDO2_3V3: track 0.00 -> 65.3 mm, vias 0 -> 5
- net VDD_ARM_SOC_IN: track 40.2 -> 104.3 mm
- net /Peripherals/LCD_ENABLE: track 0.00 -> 48.5 mm
- net /Peripherals/LCD_HSYNC: track 0.00 -> 47.8 mm, vias 0 -> 1
- net /Peripherals/LCD_CLK: track 0.00 -> 43.7 mm
- net IMX6_ONOFF: track 0.00 -> 43.7 mm, vias 0 -> 2
- net /Peripherals/LCD_VSYNC: track 0.00 -> 43.4 mm, vias 0 -> 1
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- added copper zone on In2.Cu, net /Power/VSYS
- added copper zone on In2.Cu, net LDO2_3V3
- added copper zone on F.Cu, net Net-(L1-Pad1)
- added copper zone on F.Cu, net Net-(L2-Pad1)
- added copper zone on F.Cu, net Net-(L3-Pad1)
- added copper zone on In2.Cu, net VDD_ARM_SOC_IN
- added copper zone on In2.Cu, net VSYS_5V
Other:
- board text added: "JLCJLCJLCJLC"
- board text added: "QSBC-ZERO Rev 1.0 gitlab.com/quentin-z80/qsbc-zero"
