File: peripherals.kicad_sch (KiCad schematic)
At the start: 61 parts, among them J5 Conn_02x18_Odd_Even, J8 Conn_02x16_Odd_Even, U1 MX6UL-VM

Commit message: more pcb work, bom work
Parts:
- added J?: Conn_02x18_Odd_Even, Connector_PinHeader_2.54mm:PinHeader_2x18_P2.54mm_Vertical, symbol Connector_Generic:Conn_02x18_Odd_Even
- added R22: 0R, Resistor_SMD:R_0402_1005Metric, symbol Device:R
- C53: footprint Capacitor_SMD:C_0201_0603Metric -> Capacitor_SMD:C_0402_1005Metric; DigiKey_PN (none) -> 490-14603-1-ND; MPN (none) -> GRM155R71E104KE14J; Rating 6.3V/20% -> 25V/20%
- C56: DigiKey_PN (none) -> 490-13409-1-ND; MPN (none) -> GCM155C71A105KE38D; Rating 6.3V/20% -> 10V/20%
- C80, C92: DigiKey_PN (none) -> 490-10392-1-ND; MPN (none) -> GRM033C80J224KE90D
- C81: footprint Capacitor_SMD:C_0201_0603Metric -> Capacitor_SMD:C_0402_1005Metric; DigiKey_PN (none) -> 490-12706-1-ND; MPN (none) -> GRM155R71A224KE01D; Rating 6.3V/20% -> 10V/20%
- D1: value LED -> LED_GREEN; DigiKey_PN (none) -> 511-1578-1-ND; MPN (none) -> SML-D12M8WT86
- D2: value LED -> LED_ORANGE; DigiKey_PN (none) -> 511-1583-1-ND; MPN (none) -> SML-E12D8WT86
- J5: DigiKey_PN (none) -> S2011EC-18-ND; MPN (none) -> PRPC018DAAN-RC
- J8: DigiKey_PN (none) -> S2011EC-16-ND; MPN (none) -> PRPC016DAAN-RC
- R100, R101, R102, R103, R104, R105, R106, R107, R108, R109, R62, R63, R64, R65, R66, R67, R68, R69, R70, R71, R72, R73, R74, R75, R76, R77, R78, R79, R80, R81, R82, R83, R84, R85, R86, R87, R88, R89, R90, R91, R92, R93, R94, R95, R96, R97, R98, R99: DigiKey_PN (none) -> 311-10KJRCT-ND; MPN (none) -> RC0402JR-0710KL
- R128, R129: DigiKey_PN (none) -> 311-1.0KJRCT-ND; MPN (none) -> RC0402JR-071KL
- R130: DigiKey_PN (none) -> 311-0.0LRCT-ND; MPN (none) -> RC0402FR-070RL
- U1: DigiKey_PN (none) -> 568-14995-ND; MPN (none) -> MCIMX6Y2DVM09AB
Connections:
- net DCDC_3V3: now also J5.34 (Pin_34), J5.36 (Pin_36); no longer J5.2 (Pin_2), J5.4 (Pin_4)
- net GND: now also J5.1 (Pin_1), J5.11 (Pin_11), J5.12 (Pin_12), J5.2 (Pin_2), J5.25 (Pin_25), J5.26 (Pin_26), J5.31 (Pin_31); no longer J5.15 (Pin_15), J5.16 (Pin_16), J5.29 (Pin_29), J5.30 (Pin_30), J5.35 (Pin_35), J5.5 (Pin_5), J5.6 (Pin_6)
- net GPIO1_IO03: now also J5.9 (Pin_9); no longer J5.13 (Pin_13)
- net GPIO1_IO04: now also J5.6 (Pin_6); no longer J5.10 (Pin_10)
- net GPIO1_IO05: now also J5.7 (Pin_7); no longer J5.11 (Pin_11)
- net GPIO1_IO06: now also J5.10 (Pin_10); no longer J5.14 (Pin_14)
- net GPIO1_IO07: now also J5.8 (Pin_8); no longer J5.12 (Pin_12)
- net GPIO1_IO08: now also J5.5 (Pin_5); no longer J5.9 (Pin_9)
- net GPIO1_IO09: now also J5.23 (Pin_23); no longer J5.27 (Pin_27)
- net GPIO1_IO10: now also J5.24 (Pin_24); no longer J5.28 (Pin_28)
- net GPIO1_IO11: now also J5.20 (Pin_20); no longer J5.24 (Pin_24)
- net GPIO1_IO12: now also J5.4 (Pin_4); no longer J5.8 (Pin_8)
- net GPIO1_IO13: now also J5.21 (Pin_21); no longer J5.25 (Pin_25)
- net GPIO1_IO14: now also J5.22 (Pin_22); no longer J5.26 (Pin_26)
- net GPIO1_IO15: now also J5.3 (Pin_3); no longer J5.7 (Pin_7)
- net GPIO1_IO20: now also J5.14 (Pin_14); no longer J5.18 (Pin_18)
- net GPIO1_IO21: now also J5.13 (Pin_13); no longer J5.17 (Pin_17)
- net GPIO1_IO22: now also J5.27 (Pin_27); no longer J5.31 (Pin_31)
- net GPIO1_IO23: now also J5.29 (Pin_29); no longer J5.33 (Pin_33)
- net GPIO1_IO24: now also J5.16 (Pin_16); no longer J5.20 (Pin_20)
- net GPIO1_IO25: now also J5.15 (Pin_15); no longer J5.19 (Pin_19)
- net GPIO1_IO26: now also J5.28 (Pin_28); no longer J5.32 (Pin_32)
- net GPIO1_IO27: now also J5.30 (Pin_30); no longer J5.34 (Pin_34)
- net GPIO1_IO28: now also J5.18 (Pin_18); no longer J5.22 (Pin_22)
- net GPIO1_IO29: now also J5.17 (Pin_17); no longer J5.21 (Pin_21)
- net GPIO1_IO30: now also J5.19 (Pin_19); no longer J5.23 (Pin_23)
- net GPIO1_IO31: now also J5.32 (Pin_32); no longer J5.36 (Pin_36)
- net VSYS_5V: now also J5.33 (Pin_33), J5.35 (Pin_35); no longer J5.1 (Pin_1), J5.3 (Pin_3)
- net SD1_CD_R: now reaches U1.D3 (CSI_DATA05)
- net SD1_CD_R: now also R22.1
- new net SD1_CD: R22.2
- no-connect marks 15 -> 14
Other:
- moved on the sheet: D2, R129

Commit message: add basic readme, rev 1 of pcb
Parts:
- removed J8: Conn_02x16_Odd_Even, Connector_PinHeader_2.54mm:PinHeader_2x16_P2.54mm_Vertical, symbol Connector_Generic:Conn_02x16_Odd_Even
- added D3: LED_YELLOW, LED_SMD:LED_0603_1608Metric, symbol Device:LED
- added R26: 1K, Resistor_SMD:R_0402_1005Metric, symbol Device:R
- added TP6: TestPoint, TestPoint:TestPoint_Pad_D1.0mm, symbol Connector:TestPoint
- C53: value 0.1uF -> 0.22uF; footprint Capacitor_SMD:C_0402_1005Metric -> Capacitor_SMD:C_0201_0603Metric; DigiKey_PN 490-14603-1-ND -> 490-10392-1-ND; MPN GRM155R71E104KE14J -> GRM033C80J224KE90D; Rating 25V/20% -> 6.3V/20%
- gave numbers to parts that had none: 1
Connections:
- net BT_CFG1[0]: now also J10.7 (Pin_7)
- net BT_CFG1[1]: now also J10.8 (Pin_8)
- net BT_CFG1[2]: now also J10.9 (Pin_9)
- net BT_CFG1[3]: now also J10.10 (Pin_10)
- net BT_CFG1[4]: now also J10.11 (Pin_11)
- net BT_CFG1[5]: now also J10.12 (Pin_12)
- net BT_CFG1[6]: now also J10.13 (Pin_13)
- net BT_CFG1[7]: now also J10.14 (Pin_14)
- net BT_CFG2[0]: now also J10.15 (Pin_15)
- net BT_CFG2[1]: now also J10.17 (Pin_17)
- net BT_CFG2[2]: now also J10.21 (Pin_21)
- net BT_CFG2[3]: now also J10.23 (Pin_23)
- net BT_CFG2[4]: now also J10.25 (Pin_25)
- net BT_CFG2[5]: now also J10.27 (Pin_27)
- net BT_CFG2[6]: now also J10.29 (Pin_29)
- net BT_CFG2[7]: now also J10.31 (Pin_31)
- net BT_CFG4[0]: now also J10.16 (Pin_16)
- net BT_CFG4[1]: now also J10.18 (Pin_18)
- net BT_CFG4[2]: now also J10.22 (Pin_22)
- net BT_CFG4[3]: now also J10.24 (Pin_24)
- net BT_CFG4[4]: now also J10.26 (Pin_26)
- net BT_CFG4[5]: now also J10.28 (Pin_28)
- net BT_CFG4[6]: now also J10.30 (Pin_30)
- net BT_CFG4[7]: now also J10.32 (Pin_32)
- net DCDC_3V3: now also J10.35 (Pin_35), R26.1; no longer C53.1, C56.1, U1.L13 (VDDA_ADC_3P3), U1.M13 (ADC_VREFH)
- net GND: now also J10.19 (Pin_19), J10.20 (Pin_20), J10.33 (Pin_33), J10.34 (Pin_34), J10.5 (Pin_5), J10.6 (Pin_6)
- net SD1_VSELECT: now also TP6.1
- net VSYS_5V: now also J10.36 (Pin_36)
- net LED_2: now reaches U1.D2 (CSI_DATA06)
- net LED_2: now also D3.1 (K)
- net I2C2_SDA: now reaches U1.F2 (CSI_VSYNC)
- net I2C2_SCL: now reaches U1.F3 (CSI_HSYNC)
- net LCD_CLK: now reaches U1.A8 (LCD_CLK)
- net LCD_CLK: now also J10.1 (Pin_1)
- net LCD_ENABLE: now reaches U1.B8 (LCD_ENABLE)
- net LCD_ENABLE: now also J10.2 (Pin_2)
- net LCD_VSYNC: now reaches U1.C9 (LCD_VSYNC)
- net LCD_VSYNC: now also J10.3 (Pin_3)
- net LCD_HSYNC: now reaches U1.D9 (LCD_HSYNC)
- net LCD_HSYNC: now also J10.4 (Pin_4)
- new net: D3.2 (A), R26.2
- new net LDO2_3V3: C53.1, C56.1, U1.L13 (VDDA_ADC_3P3), U1.M13 (ADC_VREFH)
- no-connect marks 14 -> 7
Other:
- moved on the sheet: J10

Commit message: misc fixes, add pics of board
Changed lines of the file:
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@@
   (symbol (lib_id "Device:R") (at 236.22 181.61 0) (unit 1)
     (in_bom yes) (on_board yes)
-    (property "Reference" "R108" (id 0) (at 234.95 187.96 90)
+    (property "Reference" "R108" (id 0) (at 234.95 189.23 90)
       (effects (font (size 1.27 1.27)) (justify left))
     )
@@
   (symbol (lib_id "Device:R") (at 220.98 181.61 0) (unit 1)
     (in_bom yes) (on_board yes)
-    (property "Reference" "R102" (id 0) (at 219.71 187.96 90)
+    (property "Reference" "R102" (id 0) (at 219.71 189.23 90)
       (effects (font (size 1.27 1.27)) (justify left))
     )
@@
   (symbol (lib_id "Device:R") (at 226.06 257.81 180) (unit 1)
     (in_bom yes) (on_board yes)
-    (property "Reference" "R105" (id 0) (at 227.33 251.46 90)
+    (property "Reference" "R105" (id 0) (at 227.33 250.19 90)
       (effects (font (size 1.27 1.27)) (justify left))
     )
@@
   (symbol (lib_id "Device:R") (at 236.22 257.81 180) (unit 1)
     (in_bom yes) (on_board yes)
-    (property "Reference" "R109" (id 0) (at 237.49 251.46 90)
+    (property "Reference" "R109" (id 0) (at 237.49 250.19 90)
       (effects (font (size 1.27 1.27)) (justify left))
     )
@@
   (symbol (lib_id "Device:R") (at 220.98 257.81 180) (unit 1)
     (in_bom yes) (on_board yes)
-    (property "Reference" "R103" (id 0) (at 222.25 251.46 90)
+    (property "Reference" "R103" (id 0) (at 222.25 250.19 90)
       (effects (font (size 1.27 1.27)) (justify left))
     )
@@
   (symbol (lib_id "Device:R") (at 215.9 181.61 0) (unit 1)
     (in_bom yes) (on_board yes)
-    (property "Reference" "R100" (id 0) (at 214.63 187.96 90)
+    (property "Reference" "R100" (id 0) (at 214.63 189.23 90)
       (effects (font (size 1.27 1.27)) (justify left))
     )
@@
   (symbol (lib_id "Device:R") (at 231.14 181.61 0) (unit 1)
     (in_bom yes) (on_board yes)
-    (property "Reference" "R106" (id 0) (at 229.87 187.96 90)
+    (property "Reference" "R106" (id 0) (at 229.87 189.23 90)
       (effects (font (size 1.27 1.27)) (justify left))
     )
@@
   (symbol (lib_id "Device:R") (at 226.06 181.61 0) (unit 1)
     (in_bom yes) (on_board yes)
-    (property "Reference" "R104" (id 0) (at 224.79 187.96 90)
+    (property "Reference" "R104" (id 0) (at 224.79 189.23 90)
       (effects (font (size 1.27 1.27)) (justify left))
     )
@@
   (symbol (lib_id "Device:R") (at 215.9 257.81 180) (unit 1)
     (in_bom yes) (on_board yes)
-    (property "Reference" "R101" (id 0) (at 217.17 251.46 90)
+    (property "Reference" "R101" (id 0) (at 217.17 250.19 90)
       (effects (font (size 1.27 1.27)) (justify left))
     )
@@
   (symbol (lib_id "Device:R") (at 231.14 257.81 180) (unit 1)
     (in_bom yes) (on_board yes)
-    (property "Reference" "R107" (id 0) (at 232.41 251.46 90)
-      (effects (font (size 1.27 1.27)) (justify left))
-    )
+    (property "Reference" "R107" (id 0) (at 232.41 250.19 90)
+      (effects (font (size 1.27 1.27)) (justify left))
+    )

Commit message: misc rev2 fixes
Parts:
- C81: footprint Capacitor_SMD:C_0402_1005Metric -> Capacitor_SMD:C_0201_0603Metric; DigiKey_PN 490-12706-1-ND -> 490-10392-1-ND; MPN GRM155R71A224KE01D -> GRM033C80J224KE90D; Rating 10V/20% -> 6.3V/20%
Changed lines of the file:
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@@
+    (pin "2")
+  )
+  (symbol (lib_id "Device:C") (at 143.51 46.99 0) (unit 1)
+    (in_bom yes) (on_board yes)
+    (property "Reference" "C81" (id 0) (at 147.32 45.7199 0)
+      (effects (font (size 1.27 1.27)) (justify left))
+    )
+    (property "Value" "0.22uF" (id 1) (at 147.32 48.2599 0)
+      (effects (font (size 1.27 1.27)) (justify left))
+    )
+    (property "Footprint" "Capacitor_SMD:C_0201_0603Metric" (id 2) (at 144.4752 50.8 0)
+      (effects (font (size 1.27 1.27)) hide)
+    )
+    (property "Datasheet" "~" (id 3) (at 143.51 46.99 0)
+      (effects (font (size 1.27 1.27)) hide)
+    )
+    (property "Rating" "6.3V/20%" (id 4) (at 148.59 50.8 0)
+      (effects (font (size 0.762 0.762)))
+    )
+    (property "DigiKey_PN" "490-10392-1-ND" (id 5) (at 143.51 46.99 0)
+      (effects (font (size 1.27 1.27)) hide)
+    )
+    (property "MPN" "GRM033C80J224KE90D" (id 6) (at 143.51 46.99 0)
+      (effects (font (size 1.27 1.27)) hide)
+    )
+    (pin "1")
     (pin "2")
   )
@@
       (effects (font (size 1.27 1.27)) hide)
     )
-    (pin "1")
-    (pin "2")
-  )
-  (symbol (lib_id "Device:C") (at 143.51 46.99 0) (unit 1)
-    (in_bom yes) (on_board yes)
-    (property "Reference" "C81" (id 0) (at 147.32 45.7199 0)
-      (effects (font (size 1.27 1.27)) (justify left))
-    )
-    (property "Value" "0.22uF" (id 1) (at 147.32 48.2599 0)
-      (effects (font (size 1.27 1.27)) (justify left))
-    )
-    (property "Footprint" "Capacitor_SMD:C_0402_1005Metric" (id 2) (at 144.4752 50.8 0)
-      (effects (font (size 1.27 1.27)) hide)
-    )
-    (property "Datasheet" "~" (id 3) (at 143.51 46.99 0)
-      (effects (font (size 1.27 1.27)) hide)
-    )
-    (property "Rating" "10V/20%" (id 4) (at 148.59 50.8 0)
-      (effects (font (size 0.762 0.762)))
-    )
-    (property "DigiKey_PN" "490-12706-1-ND" (id 5) (at 143.51 46.99 0)
-      (effects (font (size 1.27 1.27)) hide)
-    )
-    (property "MPN" "GRM155R71A224KE01D" (id 6) (at 143.51 46.99 0)
-      (effects (font (size 1.27 1.27)) hide)
-    )
