File: qsbc-zero.kicad_sch (KiCad schematic)
At the start: 4 parts

Commit message: lots of routing, ddr length matching done
Other:
- sheet Control ports: added GPIO1_IO[00..31], VDD_SNVS_3V3; removed ATS_STATUS
- sheet Ethernet ports: added I2C4_SCL, I2C4_SDA, ~{USB1_INT}; removed none
- sheet IMX6ULL Power ports: added none; removed LDO_3V3
- sheet Peripherals ports: added none; removed I2C1_SCL, I2C1_SDA, LDO_3V3, ~{USB1_INT}
- sheet Power ports: added none; removed LDO_1V8, LDO_3V3
- sheet Storage ports: added none; removed EMMC_1V8
- sheet VIN ports: added none; removed ATS_STATUS, DCDC_3V3, I2C_SCL, I2C_SDA

Commit message: more pcb work, bom work
Other:
- sheet Peripherals ports: added GPIO1_IO[00..31], SD1_CD, ~{USB1_INT}; removed none
- sheet Storage ports: added SD1_CD; removed none

Commit message: add basic readme, rev 1 of pcb
Parts:
- added C85, C86: 0.22uF, Capacitor_SMD:C_0201_0603Metric, symbol Device:C
Connections:
- net DCDC_3V3: now also C85.1, C86.1
- net GND: now also C85.2, C86.2
Other:
- sheet Control ports: added ONOFF, SNVS_3V, ~{PMIC_INT}, ~{POR}; removed GPIO_DVFS, SNVS_3V3, VDD_SNVS_3V3
- sheet DDR ports: added DDR_VREF; removed none
- sheet IMX6ULL Power ports: added SNVS_3V; removed SNVS_3V3
- sheet Peripherals ports: added I2C2_SCL, I2C2_SDA, LDO2_3V3; removed SD1_VSELECT, ~{USB1_INT}
- sheet Power ports: added DDR_VREF, I2C_SCL, I2C_SDA, IMX6_ONOFF, LDO2_3V3, SNVS_3V, ~{PMIC_INT}, ~{POR}; removed GPIO_DVFS, SD1_VSELECT, SNVS_3V3, VDD_SNVS_3V3
- sheet Storage ports: added I2C2_SCL, I2C2_SDA; removed none
- note added: "Stitching Caps for Layout"
