File: storage.kicad_sch (KiCad schematic)
At the start: 16 parts, among them J1 Micro_SD_Card_Det1, J11 Conn_01x09_Male, U1 MX6UL-VM, U26 TPD4EUSB30, U27 TPD4EUSB30, U8 D5V0H1B2LP, U9 W25Q512JVEIQ

Commit message: misc rev2 fixes
Parts:
- U9: DigiKey_PN W25Q512JVEIQ-ND -> W25Q32JVZPIQ-ND; MPN W25Q512JVEIQ -> W25Q32JVZPIQ
Changed lines of the file:
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@@
       (effects (font (size 1.27 1.27)) hide)
     )
-    (property "DigiKey_PN" "W25Q512JVEIQ-ND" (id 4) (at 64.77 181.61 0)
+    (property "DigiKey_PN" "W25Q32JVZPIQ-ND" (id 4) (at 64.77 181.61 0)
       (effects (font (size 1.27 1.27)) hide)
     )
-    (property "MPN" "W25Q512JVEIQ" (id 5) (at 64.77 181.61 0)
+    (property "MPN" "W25Q32JVZPIQ" (id 5) (at 64.77 181.61 0)
       (effects (font (size 1.27 1.27)) hide)
     )
