File: power.kicad_sch (KiCad schematic)
At the start: 42 parts, among them J8 Conn_01x09_Male, J9 Conn_01x02_Male, SW1 SW_Push, U2 MC32PF1510A6EP

Commit message: misc rev2 fixes
Parts:
- C22, C6, C8, C88, C9, C90, C96: Rating 6.3V/20% -> 10V/20%
Changed lines of the file:
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@@
       (effects (font (size 1.27 1.27)) hide)
     )
-    (property "Rating" "6.3V/20%" (id 4) (at 109.22 133.35 0)
+    (property "Rating" "10V/20%" (id 4) (at 109.22 133.35 0)
       (effects (font (size 0.762 0.762)))
     )
@@
       (effects (font (size 1.27 1.27)) hide)
     )
-    (property "Rating" "6.3V/20%" (id 4) (at 148.59 248.92 0)
+    (property "Rating" "10V/20%" (id 4) (at 148.59 248.92 0)
       (effects (font (size 0.762 0.762)))
     )
@@
       (effects (font (size 1.27 1.27)) hide)
     )
-    (property "Rating" "6.3V/20%" (id 4) (at 138.43 172.72 0)
+    (property "Rating" "10V/20%" (id 4) (at 138.43 172.72 0)
       (effects (font (size 0.762 0.762)))
     )
@@
       (effects (font (size 1.27 1.27)) hide)
     )
-    (property "Rating" "6.3V/20%" (id 4) (at 120.65 133.35 0)
+    (property "Rating" "10V/20%" (id 4) (at 120.65 133.35 0)
       (effects (font (size 0.762 0.762)))
     )
@@
       (effects (font (size 1.27 1.27)) hide)
     )
-    (property "Rating" "6.3V/20%" (id 4) (at 160.02 248.92 0)
+    (property "Rating" "10V/20%" (id 4) (at 160.02 248.92 0)
       (effects (font (size 0.762 0.762)))
     )
@@
       (effects (font (size 1.27 1.27)) hide)
     )
-    (property "Rating" "6.3V/20%" (id 4) (at 330.2 172.72 0)
+    (property "Rating" "10V/20%" (id 4) (at 330.2 172.72 0)
       (effects (font (size 0.762 0.762)))
     )
@@
       (effects (font (size 1.27 1.27)) hide)
     )
-    (property "Rating" "6.3V/20%" (id 4) (at 132.08 133.35 0)
-      (effects (font (size 0.762 0.762)))
-    )
+    (property "Rating" "10V/20%" (id 4) (at 132.08 133.35 0)
+      (effects (font (size 0.762 0.762)))
+    )

Commit message: fix cap PN
Parts:
- C7: DigiKey_PN 1276-1469-1-ND -> 1276-1467-1-ND; MPN CL05A225MQ5NNNC -> CL05A225MP5NSNC
Changed lines of the file:
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@@
       (effects (font (size 0.762 0.762)))
     )
-    (property "DigiKey_PN" "1276-1469-1-ND" (id 5) (at 139.7 52.07 0)
+    (property "DigiKey_PN" "1276-1467-1-ND" (id 5) (at 139.7 52.07 0)
       (effects (font (size 1.27 1.27)) hide)
     )
-    (property "MPN" "CL05A225MQ5NNNC" (id 6) (at 139.7 52.07 0)
+    (property "MPN" "CL05A225MP5NSNC" (id 6) (at 139.7 52.07 0)
       (effects (font (size 1.27 1.27)) hide)
     )
